File: pcb/gensym60_pcb.kicad_pcb (KiCad board)
At the start: 2 copper layers, 285.8 x 95.2 mm, 153 parts, among them J1 TYPE-C-31-M-12, J2 SM04B-SRSS-TB(LF)(SN), J3 SM04B-SRSS-TB(LF)(SN), J4 Conn_01x01, J5 Conn_01x01, J6 Conn_01x01, J7 Conn_01x01, SW1 SW_Push, SW10 SW_Push, SW11 SW_Push, SW12 SW_Push, SW13 SW_Push, SW14 SW_Push, SW15 SW_Push, SW16 SW_Push, SW17 SW_Push, SW18 SW_Push, SW19 SW_Push, SW2 SW_Push, SW20 SW_Push, SW21 SW_Push, SW22 SW_Push, SW23 SW_Push, SW24 SW_Push, SW25 SW_Push, SW26 SW_Push, SW27 SW_Push, SW28 SW_Push, SW29 SW_Push, SW3 SW_Push, SW30 SW_Push, SW31 SW_Push, SW32 SW_Push, SW33 SW_Push, SW34 SW_Push, SW35 SW_Push, SW36 SW_Push, SW37 SW_Push, SW38 SW_Push, SW39 SW_Push, SW4 SW_Push, SW40 SW_Push, SW41 SW_Push, SW42 SW_Push, SW43 SW_Push, SW44 SW_Push, SW45 SW_Push, SW46 SW_Push, SW47 SW_Push, SW48 SW_Push, SW49 SW_Push, SW5 SW_Push, SW50 SW_Push, SW51 SW_Push, SW52 SW_Push, SW53 SW_Push, SW54 SW_Push, SW55 SW_Push, SW56 SW_Push, SW57 SW_Push, SW58 SW_Push, SW59 SW_Push, SW6 SW_Push, SW60 SW_Push, SW61 SW_Push, SW62 SW_Push, SW7 SW_Push, SW8 SW_Push, SW9 SW_Push, U1 TPD4E05U06DQAR, U2 XC6206P332MR-G, U3 STM32F072CBT6

Commit message: feat: connect switches
Parts:
- C10, C11, C3, C4, C5, C6, C7, C9, R3: moved to B.Cu
- C8: value 10n -> 100n; moved to B.Cu
- moved U3 81.3 mm to (83.0, 95.9)
- moved U2 75.4 mm to (79.7, 88.7)
- moved R3 58.8 mm to (94.4, 121.2), turned to 180 degrees
- moved C4 58.8 mm to (86.6, 91.2), turned to 90 degrees
- moved C3 58.4 mm to (87.7, 99.6)
- moved C5 55.8 mm to (87.6, 91.2), turned to 90 degrees
- moved C6 54.9 mm to (87.1, 100.5)
- moved C7 50.9 mm to (83.1, 102.0), turned to -90 degrees
- moved C8 49.6 mm to (81.7, 101.6)
- moved C9 46.9 mm to (81.7, 102.5)
- moved C11 44.6 mm to (78.3, 91.3), turned to 180 degrees
- moved C10 43.9 mm to (78.3, 92.3), turned to 180 degrees
- moved D3 10.3 mm to (61.0, 113.3)
- turned SW3 to 180 degrees
Connections:
- U3 pad 37: unconnected-(U3-SWCLK/PA14-Pad37) -> COL7
Routing:
- net COL7: track 0.00 -> 344.6 mm
- net DP: track 130.7 -> 31.0 mm
- net DN: track 131.8 -> 33.1 mm
- net GND: track 130.7 -> 57.5 mm, vias 0 -> 3
- net +5V: track 83.9 -> 30.5 mm
- net +3V3: track 0.00 -> 35.3 mm
- net COL6: track 0.00 -> 7.40 mm
- net Net-(D3-A): track 6.05 -> 0.00 mm
- net Net-(U3-NRST): track 0.00 -> 1.62 mm
- net Net-(U3-BOOT0): track 0.00 -> 1.09 mm, vias 0 -> 1
- added copper zone on B.Cu, net GND
- added copper zone on F.Cu, net GND

Commit message: feat: add fuse and esd
Parts:
- removed BT1, BT2: MountingHole, kbd:Breakaway_Tabs
- removed J2, J3: SM04B-SRSS-TB(LF)(SN), acheron_Connectors:SM04B-SRSS-TB(LF)(SN)_mounting-reliefs
- removed J4, J5, J6, J7: Conn_01x01, random-keyboard-parts:Generic-Mounthole
- removed R2: 5.1k, Resistor_SMD:R_0402_1005Metric
- removed R3: 10k, Resistor_SMD:R_0402_1005Metric
- removed ZD1: SMF6.0A, acheron_Components:D_SOD-123
- added C12: 100n, acheron_Components:C_0402_1005Metric, B.Cu at (96.4, 72.9)
- C1, C2: moved to B.Cu
- F1: value ASMD1206-200 -> ASMD1206-050
- J1: value TYPE-C-31-M-12 -> JST-SH; footprint acheron_Connectors:USB_C_Receptacle_Hroparts_TYPE-C-31-M-12 -> Connector_JST:JST_SH_SM04B-SRSS-TB_1x04-1MP_P1.00mm_Horizontal
- R1: value 5.1k -> 10k; moved to B.Cu
- U1: value TPD4E05U06DQAR -> XC6206P332MR-G; footprint acheron_Components:USON-10_2.5x1.0mm_P0.5mm -> Package_TO_SOT_SMD:SOT-23-3
- U2: value XC6206P332MR-G -> STM32F072CBT6; footprint Package_TO_SOT_SMD:SOT-23-3 -> acheron_Components:LQFP-48_7x7mm_P0.5mm
- U3: value STM32F072CBT6 -> USBLC6-2SC6; footprint acheron_Components:LQFP-48_7x7mm_P0.5mm -> Package_TO_SOT_SMD:SOT-23-6
- moved SMDSW1 86.7 mm to (86.8, 105.1), turned to -90 degrees
- moved F1 84.2 mm to (99.2, 72.4)
- moved J1 80.7 mm to (104.8, 75.3), turned to -90 degrees
- moved U1 64.0 mm to (84.7, 76.1), turned to 90 degrees
- moved C1 60.1 mm to (84.2, 73.5), turned to 180 degrees
- moved C2 58.0 mm to (83.2, 78.6), turned to 180 degrees
- moved R1 50.2 mm to (88.2, 100.9)
- moved U3 26.4 mm to (99.4, 75.3), turned to 180 degrees
- moved D3 14.4 mm to (69.7, 101.8)
- moved D8 8.33 mm to (99.4, 88.7)
- moved U2 6.57 mm to (83.6, 94.0)
- moved C9 3.15 mm to (80.4, 99.7), turned to 180 degrees
- moved C7 2.56 mm to (84.1, 99.7), turned to 0 degrees
- moved C11 2.25 mm to (79.5, 89.4)
- moved C4 2.00 mm to (87.2, 89.3)
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Connections:
- C7 pad 1: Net-(U3-NRST) -> Net-(U2-NRST)
- R1 pad 1: Net-(J1-CC1) -> GND
- R1 pad 2: GND -> Net-(U2-BOOT0)
- SMDSW1 pad 2: Net-(U3-BOOT0) -> Net-(U2-BOOT0)
- SW3 pad 1: Net-(D3-A) -> COL0
- SW3 pad 2: COL0 -> Net-(D3-A)
- U1 pad 1: DP -> GND
- U1 pad 2: DN -> +3V3
- U1 pad 3: GND -> +5V
- U2 pad 1: GND -> +3V3
- U2 pad 2: +3V3 -> unconnected-(U2-PC13-Pad2)
- U2 pad 3: +5V -> unconnected-(U2-PC14/OSC32_IN-Pad3)
- U3 pad 1: +3V3 -> USB_DN
- U3 pad 2: unconnected-(U3-PC13-Pad2) -> GND
- U3 pad 3: unconnected-(U3-PC14/OSC32_IN-Pad3) -> USB_DP
- U3 pad 4: unconnected-(U3-PC15/OSC32_OUT-Pad4) -> MCU_DP
- U3 pad 5: unconnected-(U3-PF0/OSC_IN-Pad5) -> +5V
- U3 pad 6: unconnected-(U3-PF1/OSC_OUT-Pad6) -> MCU_DN
Routing:
- net COL6: track 7.40 -> 323.6 mm, vias 0 -> 8
- net COL5: track 0.00 -> 266.4 mm, vias 0 -> 6
- net COL4: track 0.00 -> 252.0 mm, vias 0 -> 8
- net COL3: track 0.00 -> 190.0 mm, vias 0 -> 6
- net COL2: track 0.00 -> 152.0 mm, vias 0 -> 6
- net COL1: track 0.00 -> 137.5 mm, vias 0 -> 8
- net ROW7: track 126.4 -> 262.4 mm
- net ROW9: track 224.8 -> 353.4 mm
- net COL0: track 0.00 -> 93.6 mm, vias 0 -> 8
- net ROW6: track 213.3 -> 306.7 mm
- net ROW5: track 167.3 -> 259.9 mm
- net ROW8: track 248.9 -> 325.1 mm
- net ROW4: track 227.6 -> 301.2 mm
- net ROW1: track 249.1 -> 311.8 mm
- net ROW0: track 273.2 -> 315.4 mm
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
Commit message: feat: move mcu
Parts:
- moved C1 1.84 mm to (82.5, 74.2)
- moved U1 1.84 mm to (83.0, 76.7)
- moved C2 1.83 mm to (81.5, 79.3)
- moved C10 1.30 mm to (78.9, 89.1)
- moved C11 1.30 mm to (79.5, 88.1)
- moved C3 1.30 mm to (88.2, 96.3)
- moved C4 1.30 mm to (87.2, 88.0)
- moved C5 1.30 mm to (88.2, 88.7)
- moved C6 1.30 mm to (87.6, 97.3)
- moved C7 1.30 mm to (84.1, 98.4)
- moved C8 1.30 mm to (82.3, 98.4)
- moved C9 1.30 mm to (80.4, 98.4)
- moved U2 1.30 mm to (83.6, 92.7)
Routing:
- net COL1: track 137.5 -> 161.0 mm
- net COL4: track 252.0 -> 275.2 mm
- net COL2: track 152.0 -> 171.9 mm
- net COL3: track 190.0 -> 207.8 mm
- net COL5: track 266.4 -> 283.7 mm
- net COL6: track 323.6 -> 339.4 mm
- net COL0: track 93.6 -> 103.5 mm
- net COL7: track 341.2 -> 350.8 mm
- net ROW5: track 259.9 -> 256.4 mm
- net ROW7: track 262.4 -> 259.8 mm
- net ROW6: track 306.7 -> 304.1 mm
- net Net-(U2-BOOT0): track 19.3 -> 16.9 mm
- net +5V: track 19.6 -> 21.8 mm
- net +3V3: track 57.7 -> 55.6 mm
- net ROW0: track 315.4 -> 313.3 mm
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Other:
- board size 285.8 x 95.2 mm -> 284.7 x 94.2 mm

Commit message: feat: tweak design for production
Other:
- board text added: "Gensym60 v1.0.0 by Susumu Ota"
