File: pcb/gensym60_pcb.kicad_pcb (KiCad board)
At the start: 2 copper layers, 284.7 x 94.2 mm, 143 parts, among them J1 JST-SH, SW1 SW_Push, SW10 SW_Push, SW11 SW_Push, SW12 SW_Push, SW13 SW_Push, SW14 SW_Push, SW15 SW_Push, SW16 SW_Push, SW17 SW_Push, SW18 SW_Push, SW19 SW_Push, SW2 SW_Push, SW20 SW_Push, SW21 SW_Push, SW22 SW_Push, SW23 SW_Push, SW24 SW_Push, SW25 SW_Push, SW26 SW_Push, SW27 SW_Push, SW28 SW_Push, SW29 SW_Push, SW3 SW_Push, SW30 SW_Push, SW31 SW_Push, SW32 SW_Push, SW33 SW_Push, SW34 SW_Push, SW35 SW_Push, SW36 SW_Push, SW37 SW_Push, SW38 SW_Push, SW39 SW_Push, SW4 SW_Push, SW40 SW_Push, SW41 SW_Push, SW42 SW_Push, SW43 SW_Push, SW44 SW_Push, SW45 SW_Push, SW46 SW_Push, SW47 SW_Push, SW48 SW_Push, SW49 SW_Push, SW5 SW_Push, SW50 SW_Push, SW51 SW_Push, SW52 SW_Push, SW53 SW_Push, SW54 SW_Push, SW55 SW_Push, SW56 SW_Push, SW57 SW_Push, SW58 SW_Push, SW59 SW_Push, SW6 SW_Push, SW60 SW_Push, SW61 SW_Push, SW62 SW_Push, SW7 SW_Push, SW8 SW_Push, SW9 SW_Push, U1 XC6206P332MR-G, U2 STM32F072CBT6, U3 USBLC6-2SC6

Commit message: chore: standardize gensym60 naming
Other:
- board text added: "gensym60 v1.0.0 by Susumu Ota"
- board text removed: "Gensym60 v1.0.0 by Susumu Ota"
Changed lines of the file:
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@@
 	(paper "A3")
 	(title_block
-		(title "Gensym60 PCB")
+		(title "gensym60 PCB")
 		(date "2025-11-01")
 		(rev "v1.0.0")
@@
 		(layer "Edge.Cuts")
 	)
-	(gr_text "Gensym60 v1.0.0 by Susumu Ota"
+	(gr_text "gensym60 v1.0.0 by Susumu Ota"
 		(at 88.180638 149.721016 0)
 		(layer "B.SilkS")
