File: pcb/gensym60_pcb.kicad_sch (KiCad schematic)
At the start: 0 parts

Commit message: feat: add usb-c daughter board
Parts:
- added BT1, BT2: MountingHole, kbd:Breakaway_Tabs, symbol Mechanical:MountingHole
- added C1, C2: 1u, acheron_Components:C_0402_1005Metric, symbol Device:C_Small
- added F1: ASMD1206-200, Fuse:Fuse_1206_3216Metric, symbol Device:Polyfuse
- added J1: TYPE-C-31-M-12, acheron_Connectors:USB_C_Receptacle_Hroparts_TYPE-C-31-M-12, symbol acheron_Symbols:TYPE-C-31-M12_13
- added J2: SM04B-SRSS-TB(LF)(SN), acheron_Connectors:SM04B-SRSS-TB(LF)(SN)_mounting-reliefs, symbol Connector_Generic_MountingPin:Conn_01x04_MountingPin
- added J4, J5, J6, J7: Conn_01x01, random-keyboard-parts:Generic-Mounthole, symbol Connector_Generic:Conn_01x01
- added R1, R2: 5.1k, Resistor_SMD:R_0402_1005Metric, symbol Device:R_Small
- added U1: TPD4E05U06DQAR, acheron_Components:USON-10_2.5x1.0mm_P0.5mm, symbol acheron_Symbols:TPD4E05U06DQAR
- added U2: RT9013-33GB, Package_TO_SOT_SMD:SOT-23-5, symbol Regulator_Linear:RT9013-33GB
- added ZD1: SMF6.0A, acheron_Components:D_SOD-123, symbol Device:D_Zener
Connections:
- new net: J1.A5 (CC1), R1.1
- new net: J1.B5 (CC2), R2.1
- new net +3V3: C2.1, U2.5 (VOUT)
- new net +5V: C1.1, F1.2, J2.1 (Pin_1), U2.1 (VIN), U2.3 (EN), ZD1.1 (K)
- new net DN: J1.A7 (D-), J1.B7 (D-), J2.2 (Pin_2), U1.2 (IO2), U1.5 (D2-), U1.6 (NC), U1.9 (NC)
- new net DP: J1.A6 (D+), J1.B6 (D+), J2.3 (Pin_3), U1.1 (IO1), U1.10 (NC), U1.4 (D2+), U1.7 (NC)
- new net GND: C1.2, C2.2, J1.A1 (GND), J1.B1 (GND), J1.S (SHIELD), J2.4 (Pin_4), J2.MP (MountPin), J5.1 (Pin_1), R1.2, R2.2, U1.3 (GND), U1.8 (GND), U2.2 (GND), ZD1.2 (A)
- new net VBUS: F1.1, J1.A4 (VBUS), J1.B4 (VBUS)
- no-connect marks 0 -> 5
Other:
- company: (none) -> Susumu Ota
- title: (none) -> Gensym60

Commit message: feat: add key matrix
Parts:
- added D1, D10, D11, D12, D13, D14, D15, D16, D17, D18, D19, D2, D20, D21, D22, D23, D24, D25, D26, D27, D28, D29, D3, D30, D31, D32, D33, D34, D35, D36, D37, D38, D39, D4, D40, D41, D42, D43, D44, D45, D46, D47, D48, D49, D5, D50, D51, D52, D53, D54, D55, D56, D57, D58, D59, D6, D60, D61, D62, D7, D8, D9: 1N4148W, acheron_Components:D_SOD-123, symbol Device:D_Small
- added SW1, SW10, SW11, SW12, SW13, SW14, SW15, SW16, SW17, SW18, SW19, SW2, SW20, SW21, SW22, SW23, SW24, SW25, SW26, SW27, SW28, SW29, SW3, SW30, SW31, SW32, SW33, SW34, SW35, SW36, SW37, SW38, SW39, SW4, SW40, SW41, SW42, SW43, SW44, SW45, SW46, SW47, SW48, SW49, SW5, SW50, SW51, SW52, SW53, SW54, SW55, SW56, SW57, SW58, SW59, SW6, SW60, SW61, SW62, SW7, SW8, SW9: SW_Push, kbd_SW:CherryMX_Hotswap_1u, symbol Switch:SW_Push
- added U3: STM32F072-LQFP48, acheron_Components:LQFP-48_7x7mm_P0.5mm, symbol acheron_Symbols:STM32F072-LQFP48
- J1: symbol acheron_Symbols:TYPE-C-31-M12_13 -> gensym60_parts:TYPE-C-31-M12_13
- U2: symbol Regulator_Linear:RT9013-33GB -> gensym60_parts:RT9013-33GB
- renumbered J4 to J3, J5 to J4, J6 to J5, J7 to J6
Connections:
- new net: D51.2 (A), SW51.1
- new net: D55.2 (A), SW55.2
- new net: D18.2 (A), SW18.1
- new net: D30.2 (A), SW30.2
- new net: D36.2 (A), SW36.1
- new net: D32.2 (A), SW32.1
- new net: D22.2 (A), SW22.2
- new net: D35.2 (A), SW35.1
- new net: D7.2 (A), SW7.1
- new net: D24.2 (A), SW24.1
- new net: D49.2 (A), SW49.1
- new net: D31.2 (A), SW31.2
- new net: D42.2 (A), SW42.1
- new net: D33.2 (A), SW33.1
- new net: D6.2 (A), SW6.2
- new net: D59.2 (A), SW59.1
- new net: D1.2 (A), SW1.1
- new net: D12.2 (A), SW12.2
- new net: D43.2 (A), SW43.1
- new net: D61.2 (A), SW61.1
- new net: D45.2 (A), SW45.2
- new net: D62.2 (A), SW62.2
- new net: D8.2 (A), SW8.1
- new net: D5.2 (A), SW5.1
- new net: D10.2 (A), SW10.1
- new net: D16.2 (A), SW16.1
- new net: D50.2 (A), SW50.1
- new net: D17.2 (A), SW17.1
- new net: D23.2 (A), SW23.2
- new net: D28.2 (A), SW28.2
- new net: D41.2 (A), SW41.1
- new net: D19.2 (A), SW19.1
- new net: D2.2 (A), SW2.1
- new net: D60.2 (A), SW60.1
- new net: D11.2 (A), SW11.1
- new net: D14.2 (A), SW14.2
- new net: D48.2 (A), SW48.2
- new net: D25.2 (A), SW25.1
- new net: D20.2 (A), SW20.2
- new net: D27.2 (A), SW27.1
- new net: D13.2 (A), SW13.2
- new net: D21.2 (A), SW21.2
- new net: D52.2 (A), SW52.1
- new net: D40.2 (A), SW40.2
- new net: D47.2 (A), SW47.2
- new net: D29.2 (A), SW29.2
- new net: D38.2 (A), SW38.2
- new net: D44.2 (A), SW44.1
- new net: D57.2 (A), SW57.1
- new net: D34.2 (A), SW34.1
- new net: D53.2 (A), SW53.1
- new net: D39.2 (A), SW39.2
- new net: D15.2 (A), SW15.2
- new net: D46.2 (A), SW46.2
- new net: D3.2 (A), SW3.1
- new net: D4.2 (A), SW4.1
- new net: D54.2 (A), SW54.2
- new net: D56.2 (A), SW56.2
- new net: D9.2 (A), SW9.1
- new net: D58.2 (A), SW58.1
- new net: D26.2 (A), SW26.1
- new net: D37.2 (A), SW37.2
- new net COL0: SW1.2, SW2.2, SW3.2, SW4.2, SW5.2, SW6.1
- new net COL1: SW10.2, SW11.2, SW12.1, SW13.1, SW14.1, SW15.1, SW7.2, SW8.2, SW9.2
- new net COL2: SW16.2, SW17.2, SW18.2, SW19.2, SW20.1, SW21.1, SW22.1, SW23.1
- new net COL3: SW24.2, SW25.2, SW26.2, SW27.2, SW28.1, SW29.1, SW30.1, SW31.1
- new net COL4: SW32.2, SW33.2, SW34.2, SW35.2, SW36.2, SW37.1, SW38.1, SW39.1, SW40.1
- new net COL5: SW41.2, SW42.2, SW43.2, SW44.2, SW45.1, SW46.1, SW47.1, SW48.1
- new net COL6: SW49.2, SW50.2, SW51.2, SW52.2, SW53.2, SW54.1, SW55.1, SW56.1
- new net COL7: SW57.2, SW58.2, SW59.2, SW60.2, SW61.2, SW62.1
- new net ROW0: D1.1 (K), D16.1 (K), D24.1 (K), D32.1 (K), D41.1 (K), D49.1 (K), D57.1 (K), D7.1 (K)
- new net ROW1: D12.1 (K), D20.1 (K), D28.1 (K), D37.1 (K), D45.1 (K), D54.1 (K), D6.1 (K)
- new net ROW2: D17.1 (K), D2.1 (K), D25.1 (K), D33.1 (K), D42.1 (K), D50.1 (K), D58.1 (K), D8.1 (K)
- new net ROW3: D13.1 (K), D21.1 (K), D29.1 (K), D38.1 (K), D46.1 (K), D55.1 (K)
- new net ROW4: D18.1 (K), D26.1 (K), D3.1 (K), D34.1 (K), D43.1 (K), D51.1 (K), D59.1 (K), D9.1 (K)
- new net ROW5: D14.1 (K), D22.1 (K), D30.1 (K), D39.1 (K), D47.1 (K)
- new net ROW6: D10.1 (K), D19.1 (K), D27.1 (K), D35.1 (K), D4.1 (K), D44.1 (K), D52.1 (K), D60.1 (K)
- new net ROW7: D23.1 (K), D31.1 (K), D40.1 (K), D48.1 (K)
- new net ROW8: D11.1 (K), D36.1 (K), D5.1 (K), D53.1 (K), D61.1 (K)
- new net ROW9: D15.1 (K), D56.1 (K), D62.1 (K)
- no-connect marks 5 -> 53
Other:
- moved on the sheet: BT1, BT2, J2, J3, J4, J5, J6

Commit message: feat: place switches
Parts:
- removed U2: RT9013-33GB, Package_TO_SOT_SMD:SOT-23-5, symbol gensym60_parts:RT9013-33GB
- added C10, C3, C4, C6, C7: 100n, acheron_Components:C_0402_1005Metric, symbol Device:C_Small
- added C11, C5: 4.7u, acheron_Components:C_0402_1005Metric, symbol Device:C_Small
- added C8: 10n, acheron_Components:C_0402_1005Metric, symbol Device:C_Small
- added C9: 1u, acheron_Components:C_0402_1005Metric, symbol Device:C_Small
- added J3: SM04B-SRSS-TB(LF)(SN), acheron_Connectors:SM04B-SRSS-TB(LF)(SN)_mounting-reliefs, symbol Connector_Generic_MountingPin:Conn_01x04_MountingPin
- added R3: 10k, Resistor_SMD:R_0402_1005Metric, symbol Device:R_Small
- added SMDSW1: TS-1187A-B-A-B, Button_Switch_SMD:SW_Push_1P1T_XKB_TS-1187A, symbol Switch:SW_Push
- added U2: XC6206P332MR-G, Package_TO_SOT_SMD:SOT-23-3, symbol Regulator_Linear:XC6206PxxxMR
- C1, C2: stock (none) -> 3486429; stock 20251019 3486429 -> (none)
- D1, D10, D11, D12, D13, D14, D15, D16, D17, D18, D19, D2, D20, D21, D22, D23, D24, D25, D26, D27, D28, D29, D3, D30, D31, D32, D33, D34, D35, D36, D37, D38, D39, D4, D40, D41, D42, D43, D44, D45, D46, D47, D48, D49, D5, D50, D51, D52, D53, D54, D55, D56, D57, D58, D59, D6, D60, D61, D62, D7, D8, D9: stock (none) -> 1819459; stock 20251019 1819459 -> (none)
- F1: stock (none) -> 2181; stock 20251019 2181 -> (none)
- J1: stock (none) -> 159900; stock 20251019 159900 -> (none)
- J2: stock (none) -> 3798; stock 20251019 3798 -> (none)
- R1, R2: stock (none) -> 2908544; stock 20251019 2908544 -> (none)
- SW1, SW10, SW12, SW13, SW14, SW16, SW17, SW18, SW19, SW20, SW21, SW22, SW23, SW24, SW25, SW26, SW27, SW28, SW29, SW30, SW31, SW32, SW33, SW34, SW35, SW37, SW38, SW39, SW40, SW41, SW42, SW43, SW44, SW45, SW46, SW47, SW48, SW49, SW50, SW51, SW52, SW54, SW55, SW56, SW57, SW6, SW61, SW62, SW7, SW8, SW9: stock (none) -> 107484; stock 20251019 107484 -> (none); now in the parts list
- SW11, SW15, SW5, SW53: footprint kbd_SW:CherryMX_Hotswap_1u -> kbd_SW:CherryMX_Hotswap_1.25u; stock (none) -> 107484; stock 20251019 107484 -> (none); now in the parts list
- SW2, SW58: footprint kbd_SW:CherryMX_Hotswap_1u -> kbd_SW:CherryMX_Hotswap_1.5u; stock (none) -> 107484; stock 20251019 107484 -> (none); now in the parts list
- SW3: footprint kbd_SW:CherryMX_Hotswap_1u -> kbd_SW:CherryMX_Hotswap_1.75u; stock (none) -> 107484; stock 20251019 107484 -> (none); now in the parts list
- SW36: footprint kbd_SW:CherryMX_Hotswap_1u -> kbd_SW:CherryMX_Hotswap_7u_Rev; stock (none) -> 107484; stock 20251019 107484 -> (none); now in the parts list
- SW4, SW59: footprint kbd_SW:CherryMX_Hotswap_1u -> kbd_SW:CherryMX_Hotswap_2.25u; stock (none) -> 107484; stock 20251019 107484 -> (none); now in the parts list
- SW60: footprint kbd_SW:CherryMX_Hotswap_1u -> kbd_SW:CherryMX_Hotswap_2.75u; stock (none) -> 107484; stock 20251019 107484 -> (none); now in the parts list
- U1: stock (none) -> 178845; stock 20251019 178845 -> (none)
- U3: value STM32F072-LQFP48 -> STM32F072CBT6; stock (none) -> 1889; stock 20251019 2189 -> (none)
- ZD1: stock (none) -> 3574; stock 20251019 3574 -> (none)
- renumbered J3 to J4, J4 to J5, J5 to J6, J6 to J7
Connections:
- net +3V3: now also U3.1 (VBAT), U3.24 (VDD), U3.36 (VDDIO2), U3.48 (VDD), U3.9 (VDDA), C10.1, C11.1, C3.1, C4.1, C5.1, C6.1, C8.1, C9.1, SMDSW1.1, U2.2 (VO)
- net +5V: now also J3.1 (Pin_1), U2.3 (VI)
- net DN: now also U3.32 (USB_DM/TIM1_CH4/PA11), J3.2 (Pin_2)
- net DP: now also U3.33 (USB_DP/PA12), J3.3 (Pin_3)
- net GND: now also U3.23 (VSS), U3.35 (VSS), U3.47 (VSS), U3.8 (VSSA), C10.2, C11.2, C3.2, C4.2, C5.2, C6.2, C7.2, C8.2, C9.2, J3.4 (Pin_4), J3.MP (MountPin), R3.1, U2.1 (GND)
- net at U3.44 (BOOT0): now also R3.2, SMDSW1.2
- net at U3.7 (NRST): now also C7.1
- no-connect marks 53 -> 40
Other:
- moved on the sheet: BT1, BT2, C1, C2, D1, D10, D11, D12, D13, D14, D15, D16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

Commit message: feat: connect switches
Parts:
- C8: value 10n -> 100n; LCSC PN C15195 -> C1525; MFR.Part # CL05B103KB5NNNC -> CL05B104KO5NNNC; stock 4539040 -> 19362316
Connections:
- net COL7: now also U3.37 (SWCLK/PA14)
- no-connect marks 40 -> 39
Changed lines of the file:
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@@
 	)
 	(junction
-		(at 246.38 140.97)
-		(diameter 0)
-		(color 0 0 0 0)
-	)
-	(junction
 		(at 120.65 38.1)
 		(diameter 0)
@@
 	)
 	(junction
-		(at 246.38 146.05)
-		(diameter 0)
-		(color 0 0 0 0)
-	)
-	(junction
 		(at 127 181.61)
 		(diameter 0)
@@
 	)
 	(junction
+		(at 246.38 146.05)
+		(diameter 0)
+		(color 0 0 0 0)
+	)
+	(junction
 		(at 99.06 190.5)
 		(diameter 0)
@@
 	)
 	(junction
+		(at 246.38 140.97)
+		(diameter 0)
+		(color 0 0 0 0)
+	)
+	(junction
 		(at 127 180.34)
 		(diameter 0)
@@
 	)
 	(no_connect
-		(at 186.69 53.34)
-	)
-	(no_connect
 		(at 274.32 110.49)
 	)
@@
 		)
 	)
+	(global_label "COL7"
+		(shape input)
+		(at 186.69 53.34 180)
+		(fields_autoplaced yes)
+		(effects
+			(font
+				(size 1.27 1.27)
+			)
+			(justify right)
+		)
+		(property "Intersheetrefs" "${INTERSHEET_REFS}"
+			(at 178.8667 53.34 0)
+			(effects
+				(font
+					(size 1.27 1.27)
+				)
+				(justify right)
+				(hide yes)
+			)
+		)
+	)
 	(global_label "DN"
 		(shape input)
@@
 	)
 	(symbol
+		(lib_id "Device:C_Small")
+		(at 246.38 143.51 0)
+		(unit 1)
+		(exclude_from_sim no)
+		(in_bom yes)
+		(on_board yes)
+		(dnp no)
+		(property "Reference" "C8"
+			(at 248.158 142.24 0)
+			(effects
+				(font
+					(size 1.27 1.27)
+				)
+				(justify left)
+			)
+		)
+		(property "Value" "100n"
+			(at 248.158 144.78 0)
+			(effects
+				(font
+					(size 1.27 1.27)
+				)
+				(justify left)
+			)
+		)
+		(property "Footprint" "acheron_Components:C_0402_1005Metric"
+			(at 246.38 143.51 0)
+			(effects
+				(font
+					(size 1.27 1.27)
+				)
+				(hide yes)
+			)
+		)
+		(property "Datasheet" "https://jlcpcb.com/api/file/downloadByFileSystemAccessId/8579707269996871680"
+			(at 246.38 143.51 0)
+			(effects
+				(font
+					(size 1.27 1.27)
+				)
+				(hide yes)
+			)
+		)
+		(property "Description" "100nF 16V X7R ±10% 0402 Multilayer Ceramic Capacitors MLCC - SMD/SMT ROHS"
+			(at 246.38 143.51 0)
+			(effects
+				(font
+					(size 1.27 1.27)
+				)
+				(hide yes)
+			)
+		)
+		(property "LCSC PN" "C1525"
+			(at 246.38 143.51 0)
+			(effects
+				(font
+					(size 1.27 1.27)
+				)
+				(hide yes)
+			)
+		)
+		(property "Basic" "1"
+			(at 246.38 143.51 0)
+			(effects
+				(font
+					(size 1.27 1.27)
+				)
+				(hide yes)
+			)
+		)
+		(property "Package" "0402"
+			(at 246.38 143.51 0)
+			(effects
+				(font
+					(size 1.27 1.27)
+				)
+				(hide yes)
+			)
+		)
+		(property "MFR.Part #" "CL05B104KO5NNNC"
+			(at 246.38 143.51 0)
+			(effects
+				(font
+					(size 1.27 1.27)
+				)
+				(hide yes)
+			)
+		)
+		(property "Manufacturer" "Samsung Electro-Mechanics"
+			(at 246.38 143.51 0)
+			(effects
+				(font
+					(size 1.27 1.27)
+				)
+				(hide yes)
+			)
+		)
+		(property "stock" "19362316"
+			(at 246.38 143.51 0)
+			(effects
+				(font
+					(size 1.27 1.27)
+				)
+				(hide yes)
+			)
+		)
+		(pin "2"
+		)
+		(pin "1"
+		)
+		(instances
+			(project "gensym60_pcb"
+				(path "/c1f78974-8be0-4f4e-b48d-4546b841f766"
+					(reference "C8")
+					(unit 1)
+				)
+			)
+		)
+	)
+	(symbol
 		(lib_id "power:GND")
 		(at 316.23 81.28 0)
@@
 					(unit 1)
 				)
-			)
-		)
-	)
-	(symbol
-		(lib_id "Device:C_Small")
-		(at 246.38 143.51 0)
-		(unit 1)
-		(exclude_from_sim no)
-		(in_bom yes)
-		(on_board yes)
-		(dnp no)
-		(property "Reference" "C8"
-			(at 248.158 142.24 0)
-			(effects
-				(font
-					(size 1.27 1.27)
-				)
-				(justify left)
-			)
-		)
-		(property "Value" "10n"
-			(at 248.158 144.78 0)
-			(effects
-				(font
-					(size 1.27 1.27)
-				)
-				(justify left)
-			)
-		)
-		(property "Footprint" "acheron_Components:C_0402_1005Metric"
-			(at 246.38 143.51 0)
-			(effects
-				(font
-					(size 1.27 1.27)
-				)
-				(hide yes)
-			)
-		)
-		(property "Datasheet" "https://jlcpcb.com/api/file/downloadByFileSystemAccessId/8579707307011465216"
-			(at 246.38 143.51 0)
-			(effects
-				(font
-					(size 1.27 1.27)
-				)
-				(hide yes)
-			)
-		)
-		(property "Description" "10nF 50V X7R ±10% 0402 Multilayer Ceramic Capacitors MLCC - SMD/SMT ROHS"
-			(at 246.38 143.51 0)
-			(effects
-				(font
-					(size 1.27 1.27)
-				)
-				(hide yes)
-			)
-		)
-		(property "LCSC PN" "C15195"
-			(at 246.38 143.51 0)
-			(effects
-				(font
-					(size 1.27 1.27)
-				)
-				(hide yes)
-			)
-		)
-		(property "Basic" "1"
-			(at 246.38 143.51 0)
-			(effects
-				(font
-					(size 1.27 1.27)
-				)
-				(hide yes)
-			)
-		)
-		(property "Package" "0402"
-			(at 246.38 143.51 0)
-			(effects
-				(font
-					(size 1.27 1.27)
-				)
-				(hide yes)
-			)
-		)
-		(property "MFR.Part #" "CL05B103KB5NNNC"
-			(at 246.38 143.51 0)
-			(effects
-				(font
-					(size 1.27 1.27)
-				)
-				(hide yes)
-			)
-		)
-		(property "Manufacturer" "Samsung Electro-Mechanics"
-			(at 246.38 143.51 0)
-			(effects
-				(font
-					(size 1.27 1.27)
-				)
-				(hide yes)
-			)
-		)
-		(property "stock" "4539040"
-			(at 246.38 143.51 0)
-			(effects
-				(font
-					(size 1.27 1.27)
-				)
-				(hide yes)
-			)
-		)
-		(pin "2"
-		)
-		(pin "1"
-		)
-		(instances
-			(project "gensym60_pcb"
-				(path "/c1f78974-8be0-4f4e-b48d-4546b841f766"
-					(reference "C8")
-					(unit 1)
-				)

Commit message: feat: add fuse and esd
Parts:
- removed BT1, BT2: MountingHole, kbd:Breakaway_Tabs, symbol Mechanical:MountingHole
- removed F1: ASMD1206-200, Fuse:Fuse_1206_3216Metric, symbol Device:Polyfuse
- removed J1: TYPE-C-31-M-12, acheron_Connectors:USB_C_Receptacle_Hroparts_TYPE-C-31-M-12, symbol gensym60_parts:TYPE-C-31-M12_13
- removed J2: SM04B-SRSS-TB(LF)(SN), acheron_Connectors:SM04B-SRSS-TB(LF)(SN)_mounting-reliefs, symbol Connector_Generic_MountingPin:Conn_01x04_MountingPin
- removed J4, J5, J6, J7: Conn_01x01, random-keyboard-parts:Generic-Mounthole, symbol Connector_Generic:Conn_01x01
- removed R1, R2: 5.1k, Resistor_SMD:R_0402_1005Metric, symbol Device:R_Small
- removed U1: TPD4E05U06DQAR, acheron_Components:USON-10_2.5x1.0mm_P0.5mm, symbol acheron_Symbols:TPD4E05U06DQAR
- removed ZD1: SMF6.0A, acheron_Components:D_SOD-123, symbol Device:D_Zener
- added C12: 100n, acheron_Components:C_0402_1005Metric, symbol Device:C_Small
- added F1: ASMD1206-050, Fuse:Fuse_1206_3216Metric, symbol Device:Polyfuse_Small
- added U3: USBLC6-2SC6, Package_TO_SOT_SMD:SOT-23-6, symbol Power_Protection:USBLC6-2SC6
- C1, C2, C9: stock 3486429 -> (none)
- C10, C3, C4, C6, C7, C8: stock 19362316 -> (none)
- C11, C5: stock 2307312 -> (none)
- D1, D10, D11, D12, D13, D14, D15, D16, D17, D18, D19, D2, D20, D21, D22, D23, D24, D25, D26, D27, D28, D29, D3, D30, D31, D32, D33, D34, D35, D36, D37, D38, D39, D4, D40, D41, D42, D43, D44, D45, D46, D47, D48, D49, D5, D50, D51, D52, D53, D54, D55, D56, D57, D58, D59, D6, D60, D61, D62, D7, D8, D9: stock 1819459 -> (none)
- J1: renamed from J3; value SM04B-SRSS-TB(LF)(SN) -> JST-SH; footprint acheron_Connectors:SM04B-SRSS-TB(LF)(SN)_mounting-reliefs -> Connector_JST:JST_SH_SM04B-SRSS-TB_1x04-1MP_P1.00mm_Horizontal; symbol Connector_Generic_MountingPin:Conn_01x04_MountingPin -> Connector_Generic:Conn_01x04; stock 3798 -> (none)
- R1: renamed from R3; stock 16492080 -> (none)
- SMDSW1: stock 371961 -> (none)
- SW1, SW10, SW11, SW12, SW13, SW14, SW15, SW16, SW17, SW18, SW19, SW2, SW20, SW21, SW22, SW23, SW24, SW25, SW26, SW27, SW28, SW29, SW3, SW30, SW31, SW32, SW33, SW34, SW35, SW36, SW37, SW38, SW39, SW4, SW40, SW41, SW42, SW43, SW44, SW45, SW46, SW47, SW48, SW49, SW5, SW50, SW51, SW52, SW53, SW54, SW55, SW56, SW57, SW58, SW59, SW6, SW60, SW61, SW62, SW7, SW8, SW9: stock 107484 -> (none)
- U1: renamed from U2; stock 917755 -> (none)
- U2: renamed from U3; stock 1889 -> (none)
Connections:
- net +5V: now also C12.1, F1.2, U3.5 (VBUS); no longer J1.1 (Pin_1)
- net COL0: now also SW3.1, U2.13 (PA3/TIM15_CH2/ADC_IN3); no longer SW3.2
- net COL1: now also U2.46 (SPI2_NSS/I2S2_WS/I2C1_SDA/TIM17_CH1/PB9)
- net COL2: now also U2.45 (I2C1_SCL/TIM16_CH1/PB8)
- net COL3: now also U2.43 (2C1_SDA/PB7)
- net COL4: now also U2.42 (I2C1_SCL/PB6)
- net COL5: now also U2.41 (SPI1_MOSI/I2S1_SD/TIM3_CH2/PB5)
- net COL6: now also U2.40 (SPI1_MISO/I2S1_MCK/TIM3_CH1/PB4)
- net COL7: now also U2.39 (SPI1_SCK/I2S1_CK/TIM2_CH2/PB3); no longer U2.37 (SWCLK/PA14)
- net GND: now also C12.2, U3.2 (GND); no longer J1.MP (MountPin)
- net ROW0: now also U2.20 (PB2)
- net ROW1: now also U2.21 (PB10/SPI2_SCK/I2C2_SCL/TIM2_CH3)
- net ROW2: now also U2.37 (SWCLK/PA14)
- net ROW3: now also U2.38 (PA15)
- net ROW4: now also U2.14 (PA4/TIM14_CH1/ADC_IN4)
- net ROW5: now also U2.15 (PA5/ADC_IN5/DAC_OUT2)
- net ROW6: now also U2.16 (PA6/ADC_IN6/TIM3_CH1/TIM16_CH1)
- net ROW7: now also U2.17 (PA7/TIM3_CH2/TIM14_CH1/ADC_IN7)
- net ROW8: now also U2.18 (PB0/TIM3_CH3/ADC_IN8)
- net ROW9: now also U2.19 (PB1/TIM3_CH4/TIM14_CH1/ADC_IN9)
- net VBUS: now also J1.1 (Pin_1), F1.1
- net at D3.2 (A): now also SW3.2; no longer SW3.1
- net DN renamed MCU_DN
- net MCU_DN: now also U3.6 (I/O1); no longer J1.2 (Pin_2)
- net DP renamed MCU_DP
- net MCU_DP: now also U3.4 (I/O2); no longer J1.3 (Pin_3)
- new net USB_DN: J1.2 (Pin_2), U3.1 (I/O1)
- new net USB_DP: J1.3 (Pin_3), U3.3 (I/O2)
- no-connect marks 39 -> 17
Other:
- moved on the sheet: C1, C2, D1, D10, D11, D12, D13, D14, D15, D16, D17, D18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

Commit message: feat: tweak design for production
Parts:
- SW1, SW10, SW11, SW12, SW13, SW14, SW15, SW16, SW17, SW18, SW19, SW2, SW20, SW21, SW22, SW23, SW24, SW25, SW26, SW27, SW28, SW29, SW3, SW30, SW31, SW32, SW33, SW34, SW35, SW37, SW38, SW39, SW4, SW40, SW41, SW42, SW43, SW44, SW45, SW46, SW47, SW48, SW49, SW5, SW50, SW51, SW52, SW53, SW54, SW55, SW56, SW57, SW58, SW59, SW6, SW60, SW61, SW62, SW7, SW8, SW9: FT Layer Override (none) -> bottom; FT Position Offset (none) -> -0.635,-3.81
- SW36: FT Layer Override (none) -> bottom; FT Position Offset (none) -> 0.635,3.81; FT Rotation Offset (none) -> 180
- U3: FT Rotation Offset (none) -> 90

Commit message: chore: standardize gensym60 naming
Other:
- title: Gensym60 -> gensym60
Changed lines of the file:
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@@
 	(paper "A2")
 	(title_block
-		(title "Gensym60")
+		(title "gensym60")
 		(date "2025-10-21")
 		(rev "v0.0.1")
